File: PCB/spelarö.kicad_pcb (KiCad board)
At the start: 2 copper layers, 90.6 x 72.6 mm, 8 parts, among them J1 Conn_01x14_Pin, SW1 K1-1506SN-01, U1 ESP32-S3-ZERO, U2 OTJ-5

Commit message: finished the pcb
Parts:
- removed U2: OTJ-5, footprints:toslink
- added G***: LOGO, LOGO, F.Cu at (134.9, 99.3)
- added G***: LOGO, LOGO, F.Cu at (129.8, 96.5)
- added G***: LOGO, LOGO, F.Cu at (134.8, 93.5)
- added G***: LOGO, LOGO, F.Cu at (145.2, 99.1)
- added G***: LOGO, LOGO, F.Cu at (140.0, 96.3)
- added G***: LOGO, LOGO, F.Cu at (140.1, 102.1)
- added G***: LOGO, LOGO, B.Cu at (159.5, 67.8)
- added REF**: MountingHole_2.2mm_M2_Pad_TopOnly, MountingHole:MountingHole_2.2mm_M2_Pad_TopOnly, F.Cu at (210.1, 102.8)
- added REF**: MountingHole_2.2mm_M2_Pad_TopOnly, MountingHole:MountingHole_2.2mm_M2_Pad_TopOnly, F.Cu at (129.5, 40.2)
- added REF**: MountingHole_2.2mm_M2_Pad_TopOnly, MountingHole:MountingHole_2.2mm_M2_Pad_TopOnly, F.Cu at (210.1, 40.2)
- added REF**: MountingHole_2.2mm_M2_Pad_TopOnly, MountingHole:MountingHole_2.2mm_M2_Pad_TopOnly, F.Cu at (129.5, 102.8)
- added U3: OTJ-5, footprints:toslink, B.Cu at (196.9, 46.2)
- moved C1 73.0 mm to (200.4, 53.6), turned to 0 degrees
- moved TF1 7.27 mm to (146.5, 44.9)
- moved U1 3.97 mm to (172.3, 48.2)
Connections:
- net /led renamed /blk
- C1 pad 1: GND -> +3.3V
- C1 pad 2: +3.3V -> GND
Routing:
- net GND: track 251.1 -> 209.5 mm, vias 6 -> 0
- net /toslink: track 70.7 -> 35.5 mm, vias 0 -> 2
- net +3.3V: track 142.5 -> 118.5 mm, vias 4 -> 1
- net /5: track 81.1 -> 64.5 mm
- net /sck: track 67.3 -> 79.3 mm, vias 3 -> 2
- net /blk: track 46.5 -> 56.9 mm, vias 1 -> 3
- net /2: track 64.2 -> 56.6 mm
- net /tft_dc: track 33.6 -> 39.9 mm
- net /4: track 64.4 -> 58.1 mm, vias 3 -> 1
- net /mosi: track 78.6 -> 73.7 mm, vias 5 -> 3
- net /3: track 66.6 -> 62.2 mm, vias 3 -> 1
- net /rst: track 35.8 -> 39.9 mm
- net /6: track 70.3 -> 66.9 mm, vias 10 -> 2
- net /1: track 52.4 -> 49.7 mm, vias 3 -> 1
- net /sd_cs: track 16.4 -> 18.9 mm, vias 2 -> 0
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Other:
- board text removed: "varför är du här bak och kollar"
