File: PCB/spelarö.kicad_pcb (KiCad board)
At the start: 2 copper layers, 90.6 x 72.6 mm, 19 parts, among them J1 Conn_01x14_Pin, SW1 K1-1506SN-01, U1 ESP32-S3-ZERO, U3 OTJ-5

Commit message: fixed the pcb
Parts:
- removed U1: ESP32-S3-ZERO, footprints:MODULE_ESP32-S3-ZERO
- added A1: Arduino_Nano_ESP32, footprints:MODULE_NANO-ESP32-ENTRY, B.Cu at (176.6, 58.9)
- added LED1: WS2812B, footprints:WS2812B, F.Cu at (169.8, 99.2)
- added R1: 10k, Resistor_SMD:R_1206_3216Metric, B.Cu at (145.4, 59.5)
- added R2: 10k, Resistor_SMD:R_1206_3216Metric, B.Cu at (139.0, 59.5)
- added R3: 10k, Resistor_SMD:R_1206_3216Metric, B.Cu at (131.9, 58.5)
- SW1: footprint footprints:KEY-SMD_K1-1506SN-01 -> footprints:C145910
- moved S1 5.55 mm to (183.7, 99.6)
- moved SW1 2.34 mm to (156.2, 99.0)
Connections:
- S1 pad 1: /6 -> GND
- S1 pad 2: /6 -> GND
- S1 pad 3: GND -> /6
- S1 pad 4: GND -> /6
- U3 pad 1: /toslink -> GND
- U3 pad 3: GND -> /toslink
Routing:
- net +5V: track 0.00 -> 73.4 mm, vias 0 -> 3
- net +3.3V: track 118.5 -> 171.6 mm, vias 1 -> 6
- net /sd_cs: track 18.9 -> 55.3 mm, vias 0 -> 2
- net /neopixel: track 0.00 -> 34.4 mm, vias 0 -> 3
- net /1: track 49.7 -> 83.0 mm, vias 1 -> 3
- net /5: track 64.5 -> 33.8 mm
- net /blk: track 56.9 -> 29.0 mm, vias 3 -> 1
- net /miso: track 87.1 -> 110.7 mm
- net /6: track 66.9 -> 45.5 mm, vias 2 -> 0
- net /3: track 62.2 -> 82.8 mm, vias 1 -> 5
- net GND: track 209.5 -> 189.6 mm, vias 0 -> 1
- net /mosi: track 73.7 -> 92.8 mm, vias 3 -> 2
- net /sck: track 79.3 -> 95.9 mm, vias 2 -> 8
- net /tft_cs: track 41.9 -> 27.9 mm, vias 0 -> 2
- net /toslink: track 35.5 -> 49.1 mm
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Other:
- board text added: "v3"
- board text removed: "v2"
