File: PCB/spelarö.kicad_sch (KiCad schematic)
At the start: 7 parts, among them J1 Conn_01x14_Pin, SW1 K1-1506SN-01, U1 ESP32-S3-ZERO, U2 OTJ-5

Commit message: finished the pcb
Parts:
- removed U2: OTJ-5, footprints:toslink, symbol FCR684205T:OTJ-5
- added U3: OTJ-5, footprints:toslink, symbol FCR684205T:OTJ-5
Connections:
- net +3.3V: now also C1.1, U3.2 (VCC); no longer C1.2
- net GND: now also C1.2, U3.3 (GND); no longer C1.1
- net toslink: now also U3.1 (VIN)
Other:
- moved on the sheet: C1
