File: PCB/spelarö.kicad_sch (KiCad schematic)
At the start: 7 parts, among them J1 Conn_01x14_Pin, SW1 K1-1506SN-01, U1 ESP32-S3-ZERO, U3 OTJ-5

Commit message: fixed the pcb
Parts:
- removed U1: ESP32-S3-ZERO, footprints:MODULE_ESP32-S3-ZERO, symbol ESP32-S3-ZERO:ESP32-S3-ZERO
- added A1: Arduino_Nano_ESP32, footprints:MODULE_NANO-ESP32-ENTRY, symbol MCU_Module:Arduino_Nano_ESP32
- added LED1: WS2812B, footprints:WS2812B, symbol WS2812B:WS2812B
- added R1, R2, R3: 10k, Resistor_SMD:R_1206_3216Metric, symbol Device:R
- SW1: footprint footprints:KEY-SMD_K1-1506SN-01 -> footprints:C145910
Connections:
- net +3.3V: now also A1.17 (3V3), R1.1, R2.1, R3.1
- net +5V: now also A1.27 (VUSB/5V), LED1.1-VDD (VDD)
- net 1: now also A1.5 (D2)
- net 2: now also A1.6 (D3)
- net 3: now also A1.7 (D4)
- net 4: now also A1.8 (D5)
- net 5: now also A1.14 (D11/COPI)
- net 6: now also S1.3, S1.4, A1.20 (A1); no longer S1.1, S1.2
- net GND: now also S1.1, S1.2, U3.1 (GND), A1.29 (GND), A1.4 (GND), LED1.3-GND (GND); no longer S1.3, S1.4, U3.3 (GND)
- net blk: now also A1.9 (D6)
- net miso: now also A1.24 (SCL/A5), R3.2
- net mosi: now also A1.23 (SDA/A4), R2.2
- net rst: now also A1.10 (D7)
- net sck: now also A1.16 (D13/SCK)
- net sd_cs: now also A1.13 (D10/CS), R1.2
- net tft_cs: now also A1.12 (D9)
- net tft_dc: now also A1.11 (D8)
- net toslink: now also U3.3 (VIN), A1.19 (A0); no longer U3.1 (VIN)
- new net neopixel: A1.15 (D12/CIPO), LED1.4-DIN (DI)
- no-connect marks 8 -> 19
Other:
- note added: "buttons"
- note added: "microcontroller"
- note added: "neopixel"
- note removed: "button"
- note removed: "esp32"
- moved on the sheet: C1, J1, U3

Commit message: fixed bom
Other:
- company: (none) -> konrad
- title: (none) -> spelarö
Changed lines of the file:
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@@
 	(generator_version "10.0")
 	(paper "A4")
+	(title_block
+		(title "spelarö")
+		(date "2026-08-01")
+		(rev "V1")
+		(company "konrad")
+	)
 	(rectangle
 		(start 104.14 13.97)
